Commit message: debugging

File: src/thaiquiri_webots/resource/thaiquiri.urdf (robot description, URDF)
Before this commit: robot thaiquiri, 28 links, 27 joints
Links:
- added link imu_link
Joints:
- added joint cube_orange_imu_joint: type fixed, parent cube_orange, child imu_link, origin xyz=0 0 0 rpy=-1.5707963267948966 -1.5707963267948966 0
- joint ZED_X_Mini_camera_camera_right_joint: origin xyz=0.025 0.003 0.003 rpy=0 0 0 -> xyz=0.025 0.003 0 rpy=0 0 0
